Commit message: Changed the names of the links and joint in order to keep the same standard with robcogen

File: robots/hyl_gazebo.urdf.xacro (robot description, xacro)
@@ -22,9 +22,8 @@
 	<!-- LF leg -->
 	<xacro:hyl_leg
-		name="lf"
 		parent="support"
 		reflect_upper="1"
 		reflect_front="1">
-		<origin xyz="0 0 0" rpy="0 0 0"/>
+		<origin xyz="0 0 0.85" rpy="0 0 0"/>
 	</xacro:hyl_leg>
 </robot>

File: urdfs/common_gazebo.xacro (robot description, xacro)
@@ -4,5 +4,4 @@
 	<!-- standard distances -->
 	<property name="d_lr" value="0.28"/>
-	<property name="d_fh" value="0.747"/>
 	<property name="d_tbb" value="0.0825"/>
 	<property name="d_p1p2" value="0.35"/>

File: urdfs/leg/leg.gazebo.xacro (robot description, xacro)
@@ -1,6 +1,6 @@
 <?xml version="1.0"?>
 <robot xmlns:xacro="http://www.ros.org/wiki/xacro">
-	<xacro:macro name="leg_gazebo" params="name">
-		<gazebo reference="${name}_lower_leg">
+	<xacro:macro name="leg_gazebo">
+		<gazebo reference="lowerleg">
 			<kp>1000000.0</kp>
 			<kd>100.0</kd>

File: urdfs/leg/leg.transmission.xacro (robot description, xacro)
@@ -1,12 +1,12 @@
 <?xml version="1.0"?>
 <robot xmlns:xacro="http://www.ros.org/wiki/xacro">
-	<xacro:macro name="leg_transmission" params="name">
+	<xacro:macro name="leg_transmission">
     	<!-- Slider -->
-		<transmission name="slider_z_trans">
+		<transmission name="slider_trans">
 			<type>transmission_interface/SimpleTransmission</type>
-			<joint name="slider_z_joint">
+			<joint name="slider_joint">
 				<hardwareInterface>EffortJointInterface</hardwareInterface>
 			</joint>
-			<actuator name="slider_z_motor">
+			<actuator name="slider_motor">
 				<hardwareInterface>EffortJointInterface</hardwareInterface>
 				<mechanicalReduction>1</mechanicalReduction>
@@ -14,10 +14,10 @@
 		</transmission>
     	<!-- Upper leg -->
-		<transmission name="${name}_haa_trans">
+		<transmission name="haa_trans">
 			<type>transmission_interface/SimpleTransmission</type>
-			<joint name="${name}_haa_joint">
+			<joint name="haa_joint">
 				<hardwareInterface>EffortJointInterface</hardwareInterface>
 			</joint>
-			<actuator name="${name}_haa_motor">
+			<actuator name="haa_motor">
 				<hardwareInterface>EffortJointInterface</hardwareInterface>
 				<mechanicalReduction>1</mechanicalReduction>
@@ -25,10 +25,10 @@
 		</transmission>
     	<!-- Upper leg -->
-		<transmission name="${name}_hfe_upper_trans">
+		<transmission name="hfe_upper_trans">
 			<type>transmission_interface/SimpleTransmission</type>
-			<joint name="${name}_hfe_joint">
+			<joint name="hfe_joint">
 				<hardwareInterface>EffortJointInterface</hardwareInterface>
 			</joint>
-			<actuator name="${name}_hfe_motor">
+			<actuator name="hfe_motor">
 				<hardwareInterface>EffortJointInterface</hardwareInterface>
 				<mechanicalReduction>1</mechanicalReduction>
@@ -36,10 +36,10 @@
 		</transmission>
     	<!-- Lower leg -->
-		<transmission name="${name}_kfe_trans">
+		<transmission name="kfe_trans">
 			<type>transmission_interface/SimpleTransmission</type>
-			<joint name="${name}_kfe_joint">
+			<joint name="kfe_joint">
 				<hardwareInterface>EffortJointInterface</hardwareInterface>
 			</joint>
-			<actuator name="${name}_kfe_motor">
+			<actuator name="kfe_motor">
 				<hardwareInterface>EffortJointInterface</hardwareInterface>
 				<mechanicalReduction>1</mechanicalReduction>

File: urdfs/leg/leg.urdf.xacro (robot description, xacro)
@@ -6,27 +6,26 @@
 	<!-- ================================== Leg ================================== -->
 	<!-- The xacro macro xacro:hyl_leg contains: slider upper and lower leg -->
-	<xacro:macro name="hyl_leg" params="name parent *origin reflect_upper reflect_front">
+	<xacro:macro name="hyl_leg" params="parent *origin reflect_upper reflect_front">
 		<!-- Joints -->
 		<!-- Slider joint -->
-		<joint name="slider_z_joint" type="prismatic">
+		<joint name="slider_joint" type="prismatic">
 			<insert_block name="origin"/>
 			<parent link="${parent}"/>
 			<child  link="slider"/>
-			<limit effort="1000.0" velocity="1.0" lower="-0.1" upper="0.1"/>
+			<limit effort="100000.0" velocity="100.0" lower="-0.60" upper="0.5"/>
 			<axis xyz="0 0 1"/>
 			<dynamics damping="0.1" friction="0" />
-			<safety_controller k_position="100" k_velocity="100" soft_lower_limit="-10" soft_upper_limit="12.45" />
 		</joint>
 		<!-- Hip assembly joint -->
-		<joint name="${name}_assembly_joint" type="fixed">
-			<origin xyz="0 ${-d_lr/2} 0" rpy="0 ${PI/2} ${PI}"/>
+		<joint name="assembly_joint" type="fixed">
+			<origin xyz="0 ${d_lr/2} 0" rpy="0 ${PI/2} ${PI}"/>
 			<parent link="slider"/>
-			<child  link="${name}_assembly"/>
+			<child  link="assembly"/>
 		</joint>
 		<!-- Virtual hip joint assembly -->
-		<joint name="${name}_haa_joint" type="revolute">
+		<joint name="haa_joint" type="revolute">
 			<origin xyz="0 0 0" rpy="0 0 0"/>
-			<parent link="${name}_assembly"/>
-			<child  link="${name}_virtual_assembly"/>
+			<parent link="assembly"/>
+			<child  link="hipassembly"/>
 			<limit effort="200.0" velocity="1000.0" lower="${-PI/2}" upper="${PI/6}"/>
 			<axis xyz="0 0 1"/>
@@ -35,8 +34,8 @@
 		</joint>
 		<!-- Upper leg joint -->
-		<joint name="${name}_hfe_joint" type="revolute">
+		<joint name="hfe_joint" type="revolute">
 			<origin xyz="${d_tbb} 0.0 0.0" rpy="${reflect_upper*PI/2} ${-1*hfe_pos0} 0.0"/>
-			<parent link="${name}_assembly"/>
-			<child  link="${name}_upper_leg"/>
+			<parent link="hipassembly"/>
+			<child  link="upperleg"/>
 			<limit effort="200.0" velocity="1.0" lower="${-(1+reflect_front)*5*PI/36-(1-reflect_front)*7*PI/36-reflect_front*hfe_pos0}" upper="${(1-reflect_front)*5*PI/36+(1+reflect_front)*7*PI/36-reflect_front*hfe_pos0}"/>
 			<axis xyz="0 0 1"/>
@@ -45,8 +44,8 @@
 		</joint>
 		<!-- Lower leg joint -->
-		<joint name="${name}_kfe_joint" type="revolute">
+		<joint name="kfe_joint" type="revolute">
 			<origin xyz="${d_p1p2} 0.0 0.0" rpy="0.0 0.0 ${reflect_front*kfe_pos0}"/>
-			<parent link="${name}_upper_leg"/>
-			<child  link="${name}_lower_leg"/>
+			<parent link="upperleg"/>
+			<child  link="lowerleg"/>
 			<limit effort="200.0" velocity="1.0" lower="${-(1+reflect_front)*7*PI/18+(1-reflect_front)*PI/18-reflect_front*kfe_pos0}" upper="${(1-reflect_front)*7*PI/18-(1+reflect_front)*PI/18-reflect_front*kfe_pos0}"/>
 			<axis xyz="0 0 1"/>
@@ -55,8 +54,8 @@
 		</joint>
 		<!-- Foot joint -->
-		<joint name="${name}_foot_joint" type="fixed">
+		<joint name="foot_joint" type="fixed">
 			<origin xyz="0.34 0.0 0.0" rpy="${PI/2} 0.0 ${-PI/2}"/>
-			<parent link="${name}_lower_leg"/>
-			<child  link="${name}_foot"/>
+			<parent link="lowerleg"/>
+			<child  link="foot"/>
 		</joint>
 		<!-- Links -->
@@ -69,6 +68,6 @@
 			</inertial>
 		</link>
-		<!-- Hip assembly link -->
-		<link name="${name}_assembly">
+		<!-- Leg assembly link -->
+		<link name="assembly">
 			<inertial>
 				<origin xyz="0.0 0.0 0.0"/>
@@ -77,6 +76,6 @@
 			</inertial>
 		</link>
-		<!-- Virtual hip assembly link -->
-		<link name="${name}_virtual_assembly">
+		<!-- Hip assembly link -->
+		<link name="hipassembly">
 			<inertial>
 				<origin xyz="0.0 0.0 0.0"/>
@@ -86,5 +85,5 @@
 		</link>
 		<!-- Upper leg link -->
-		<link name="${name}_upper_leg">
+		<link name="upperleg">
 			<inertial>
 				<origin xyz="0.14796 ${reflect_upper*0.02958} 0.0"/>
@@ -106,5 +105,5 @@
 		</link>
 		<!-- Lower leg link -->
-		<link name="${name}_lower_leg">
+		<link name="lowerleg">
 			<inertial>
 				<origin xyz=" 0.17830  0.00030 -0.00010"/>
@@ -125,5 +124,5 @@
 		</link>
 		<!-- Foot link -->
-		<link name="${name}_foot">
+		<link name="foot">
 			<inertial>
 				<origin xyz="0.0 0.0 0.0"/>
@@ -145,6 +144,6 @@
 		</link>
 		<!-- Extensions -->
-		<xacro:leg_transmission name="${name}"/>
-		<xacro:leg_gazebo name="${name}"/>
+		<xacro:leg_transmission/>
+		<xacro:leg_gazebo/>
 	</xacro:macro>
 </robot>

File: urdfs/support/support.urdf.xacro (robot description, xacro)
@@ -2,5 +2,4 @@
 <robot xmlns:xacro="http://www.ros.org/wiki/xacro">
 	<!-- Things that are needed only for Gazebo (not the physical robot). These include sensor and controller plugin specifications -->
-<!--	<xacro:include filename="$(find hyl_description)/urdfs/trunk/support.gazebo.xacro"/>-->
 	<!-- =============================== Support =============================== -->
 	<!-- The xacro macro xacro:hyl_support contains: support of HyL -->
@@ -8,5 +7,5 @@
 		<!-- Floating-base Joint -->
 		<joint name="support_joint" type="fixed">
-			<origin xyz="0 0 0.85" rpy="0 0 0"/>
+			<origin xyz="0 0 0" rpy="0 0 0"/>
 			<parent link="${name}_link"/>
 			<child link="support"/>
@@ -24,10 +23,10 @@
 		<link name="support">
 			<inertial>
-				<origin xyz="0 0 -0.575"/>
+				<origin xyz="0 0 0"/>
 				<mass value="5000"/>
 				<inertia ixx="25000" iyy="25000" izz="25000" ixy="0" ixz="0" iyz="0"/>
 			</inertial>
 			<collision>
-				<origin xyz="0 0 -0.575" rpy="0 0 0" />
+				<origin xyz="0 0 0.575" rpy="0 0 0" />
 				<geometry>
 					<box size="0.12 0.045 1.15" />
@@ -36,5 +35,5 @@
 			</collision>
 			<visual>
-				<origin xyz="0 0 -0.575" rpy="0 0 0" />
+				<origin xyz="0 0 0.575" rpy="0 0 0" />
 				<geometry>
 					<box size="0.12 0.045 1.15" />
@@ -43,6 +42,4 @@
 			</visual>
 		</link>
-		<!-- Extensions -->
-<!--		<xacro:trunk_gazebo name="trunk"/>-->
 	</xacro:macro>
 </robot>
