Commit message: Removed the label that changes angles because these aren't necessaries for one leg

File: robots/hyl.urdf.xacro (robot description, xacro)
@@ -20,9 +20,6 @@
 	<!-- trunk -->
 	<xacro:hyl_support name="base" />
-	<!-- LF leg -->
-	<xacro:hyl_leg
-		parent="support"
-		reflect_upper="1"
-		reflect_front="1">
+	<!-- leg -->
+	<xacro:hyl_leg parent="support">
 		<origin xyz="0 0 0.85" rpy="0 0 0"/>
 	</xacro:hyl_leg>

File: urdfs/leg/leg.urdf.xacro (robot description, xacro)
@@ -6,5 +6,5 @@
 	<!-- ================================== Leg ================================== -->
 	<!-- The xacro macro xacro:hyl_leg contains: slider upper and lower leg -->
-	<xacro:macro name="hyl_leg" params="parent *origin reflect_upper reflect_front">
+	<xacro:macro name="hyl_leg" params="parent *origin">
 		<!-- Joints -->
 		<!-- Slider joint -->
@@ -35,9 +35,9 @@
 		<!-- Upper leg joint -->
 		<joint name="hfe_joint" type="revolute">
-			<origin xyz="${d_tbb} 0 0" rpy="${reflect_upper*PI/2} 0 0"/>
+			<origin xyz="${d_tbb} 0 0" rpy="${PI/2} 0 0"/>
 			<parent link="hipassembly"/>
 			<child  link="upperleg"/>
-			<limit effort="200.0" velocity="1.0" lower="${-(1+reflect_front)*5*PI/36-(1-reflect_front)*7*PI/36}"
-				   upper="${(1-reflect_front)*5*PI/36+(1+reflect_front)*7*PI/36}"/>
+			<limit effort="200.0" velocity="1.0" lower="${-10*PI/36}"
+				   upper="${14*PI/36}"/>
 			<axis xyz="0 0 1"/>
 			<dynamics damping="0.1" friction="0" />
@@ -49,6 +49,6 @@
 			<parent link="upperleg"/>
 			<child  link="lowerleg"/>
-			<limit effort="200.0" velocity="1.0" lower="${-(1+reflect_front)*7*PI/18+(1-reflect_front)*PI/18}"
-				   upper="${(1-reflect_front)*7*PI/18-(1+reflect_front)*PI/18}"/>
+			<limit effort="200.0" velocity="1.0" lower="${-14*PI/18}"
+				   upper="${-2*PI/18}"/>
 			<axis xyz="0 0 1"/>
 			<dynamics damping="0.1" friction="0" />
@@ -90,5 +90,5 @@
 		<link name="upperleg">
 			<inertial>
-				<origin xyz="${xcom_upperleg} ${reflect_upper*ycom_upperleg} ${zcom_upperleg}"/>
+				<origin xyz="${xcom_upperleg} ${ycom_upperleg} ${zcom_upperleg}"/>
 				<mass value="${m_upperleg}"/>
 				<inertia ixx="${ixx_upperleg}" iyy="${iyy_upperleg}" izz="${izz_upperleg}"
@@ -96,5 +96,5 @@
 			</inertial>
 			<visual>
-				<origin xyz="0 0 0" rpy="${(1-reflect_front)*PI/2} 0 0"/>
+				<origin xyz="0 0 0" rpy="0 0 0"/>
 				<geometry>
 					<mesh filename="package://hyl_description/meshes/leg/upper.dae" scale="1 1 1"/>
@@ -102,5 +102,5 @@
 			</visual>
 			<collision>
-				<origin xyz="0 0 0" rpy="${(1-reflect_front)*PI/2} 0 0"/>
+				<origin xyz="0 0 0" rpy="0 0 0"/>
 				<geometry>
 					<mesh filename="package://hyl_description/meshes/leg/upper.dae" scale="1 1 1"/>

Commit message: Removed an useless joint

File: robots/hyl.urdf.xacro (robot description, xacro)
@@ -19,7 +19,7 @@
 	<!-- body -->
 	<!-- trunk -->
-	<xacro:hyl_support name="base" />
+	<xacro:hyl_support/>
 	<!-- leg -->
-	<xacro:hyl_leg parent="support">
+	<xacro:hyl_leg parent="base_link">
 		<origin xyz="0 0 0.85" rpy="0 0 0"/>
 	</xacro:hyl_leg>

File: urdfs/support/support.urdf.xacro (robot description, xacro)
@@ -4,22 +4,6 @@
 	<!-- =============================== Support =============================== -->
 	<!-- The xacro macro xacro:hyl_support contains: support of HyL -->
-	<xacro:macro name="hyl_support" params="name">
-		<!-- Floating-base Joint -->
-		<joint name="support_joint" type="fixed">
-			<origin xyz="0 0 0" rpy="0 0 0"/>
-			<parent link="${name}_link"/>
-			<child link="support"/>
-		</joint>
-		<!-- Links -->
-		<!-- Footprint link -->
-		<link name="${name}_link">
-			<visual>
-				<geometry>
-					<cylinder length="0.01" radius="0.01"/>
-				</geometry>
-			</visual>
-		</link>
-		<!-- Trunk link -->
-		<link name="support">
+	<xacro:macro name="hyl_support">
+		<link name="base_link">
 			<inertial>
 				<origin xyz="0 0 0"/>

Commit message: Removed the dynamic of the support

File: robots/hyl.urdf.xacro (robot description, xacro)
@@ -17,7 +17,7 @@
 the origin block defines where the component is w.r.t its parent (in this case the parent
 is the world frame). For more, see http://www.ros.org/wiki/xacro -->
-	<!-- body -->
-	<!-- trunk -->
-	<xacro:hyl_support/>
+	<!-- support -->
+	<link name="world"/>
+	<xacro:hyl_support parent="world"/>
 	<!-- leg -->
 	<xacro:hyl_leg parent="base_link">

File: urdfs/support/support.urdf.xacro (robot description, xacro)
@@ -4,10 +4,15 @@
 	<!-- =============================== Support =============================== -->
 	<!-- The xacro macro xacro:hyl_support contains: support of HyL -->
-	<xacro:macro name="hyl_support">
+	<xacro:macro name="hyl_support" params="parent">
+		<joint name="${parent}_joint" type="fixed">
+			<parent link="${parent}"/>
+			<child link="base_link"/>
+			<origin rpy="0 0 0" xyz="0 0 0"/>
+		</joint>
 		<link name="base_link">
 			<inertial>
 				<origin xyz="0 0 0"/>
-				<mass value="5000"/>
-				<inertia ixx="25000" iyy="25000" izz="25000" ixy="0" ixz="0" iyz="0"/>
+				<mass value="0.1"/>
+				<inertia ixx="0.01" iyy="0.01" izz="0.01" ixy="0" ixz="0" iyz="0"/>
 			</inertial>
 			<collision>

Commit message: Adding a proper displacement in y

File: robots/hyl.urdf.xacro (robot description, xacro)
@@ -22,5 +22,5 @@
 	<!-- leg -->
 	<xacro:hyl_leg parent="base_link">
-		<origin xyz="0 0 0.85" rpy="0 0 0"/>
+		<origin xyz="0 0.025 0.85" rpy="0 0 0"/>
 	</xacro:hyl_leg>
 </robot>

Commit message: Aligned the base_link with the trunk link. This is a more clear representation

File: robots/hyl.urdf.xacro (robot description, xacro)
@@ -22,5 +22,5 @@
 	<!-- leg -->
 	<xacro:hyl_leg parent="base_link">
-		<origin xyz="0 0.025 0.85" rpy="0 0 0"/>
+		<origin xyz="0 0 0" rpy="0 0 0"/>
 	</xacro:hyl_leg>
 </robot>

File: urdfs/support/support.urdf.xacro (robot description, xacro)
@@ -8,5 +8,5 @@
 			<parent link="${parent}"/>
 			<child link="base_link"/>
-			<origin rpy="0 0 0" xyz="0 0 0"/>
+			<origin xyz="0 0.025 0.85" rpy="0 0 0"/>
 		</joint>
 		<link name="base_link">
@@ -17,5 +17,5 @@
 			</inertial>
 			<collision>
-				<origin xyz="0 0 0.575" rpy="0 0 0" />
+				<origin xyz="0 -0.025 -0.275" rpy="0 0 0" />
 				<geometry>
 					<box size="0.12 0.045 1.15" />
@@ -23,5 +23,5 @@
 			</collision>
 			<visual>
-				<origin xyz="0 0 0.575" rpy="0 0 0" />
+				<origin xyz="0 -0.025 -0.275" rpy="0 0 0" />
 				<geometry>
 					<box size="0.12 0.045 1.15" />

Commit message: [feature] Added the internal_wrench sensor

File: robots/hyl.urdf.xacro (robot description, xacro)
@@ -1,4 +1,6 @@
 <?xml version="1.0"?>
 <robot name="hyl" xmlns:xacro="http://www.ros.org/wiki/xacro">
+	<!-- This argument allows us to load joint sensors that measure the internal wrenches -->
+	<xacro:arg name="load_force_sensors" default="false"/>
 	<!-- The following included files set up definitions of parts of the robot body -->
 	<xacro:include filename="$(find hyl_description)/urdfs/common.xacro"/>
@@ -21,5 +23,5 @@
 	<xacro:hyl_support parent="world"/>
 	<!-- leg -->
-	<xacro:hyl_leg parent="base_link">
+	<xacro:hyl_leg parent="base_link" load_force_sensors="$(arg load_force_sensors)">
 		<origin xyz="0 0 0" rpy="0 0 0"/>
 	</xacro:hyl_leg>

File: urdfs/leg/leg.gazebo.xacro (robot description, xacro)
@@ -1,5 +1,44 @@
 <?xml version="1.0"?>
 <robot xmlns:xacro="http://www.ros.org/wiki/xacro">
-	<xacro:macro name="leg_gazebo">
+	<xacro:macro name="leg_gazebo" params="load_force_sensors">
+		<gazebo reference="slider_joint">
+			<provideFeedback>true</provideFeedback>
+		</gazebo>
+		<xacro:if value="${load_force_sensors}">
+			<gazebo>
+				<plugin name="slider_sensor" filename="libgazebo_ros_ft_sensor.so">
+					<robotNamespace>/hyl/internal_wrench/</robotNamespace>
+					<updateRate>100.0</updateRate>
+					<topicName>slider_joint</topicName>
+					<jointName>slider_joint</jointName>
+				</plugin>
+			</gazebo>
+		</xacro:if>
+		<gazebo reference="kfe_joint">
+			<provideFeedback>true</provideFeedback>
+		</gazebo>
+		<xacro:if value="${load_force_sensors}">
+			<gazebo>
+				<plugin name="kfe_sensor" filename="libgazebo_ros_ft_sensor.so">
+					<robotNamespace>/hyl/internal_wrench/</robotNamespace>
+					<updateRate>100.0</updateRate>
+					<topicName>kfe_joint</topicName>
+					<jointName>kfe_joint</jointName>
+				</plugin>
+			</gazebo>
+		</xacro:if>
+		<gazebo reference="hfe_joint">
+			<provideFeedback>true</provideFeedback>
+		</gazebo>
+		<xacro:if value="${load_force_sensors}">
+			<gazebo>
+				<plugin name="hfe_sensor" filename="libgazebo_ros_ft_sensor.so">
+					<robotNamespace>/hyl/internal_wrench/</robotNamespace>
+					<updateRate>100.0</updateRate>
+					<topicName>hfe_joint</topicName>
+					<jointName>hfe_joint</jointName>
+				</plugin>
+			</gazebo>
+		</xacro:if>
 		<gazebo reference="foot">
 			<kp>1000000.0</kp>

File: urdfs/leg/leg.urdf.xacro (robot description, xacro)
@@ -6,5 +6,5 @@
 	<!-- ================================== Leg ================================== -->
 	<!-- The xacro macro xacro:hyl_leg contains: slider upper and lower leg -->
-	<xacro:macro name="hyl_leg" params="parent *origin">
+	<xacro:macro name="hyl_leg" params="parent *origin load_force_sensors">
 		<!-- Joints -->
 		<!-- Slider joint -->
@@ -151,5 +151,5 @@
 		<!-- Extensions -->
 		<xacro:leg_transmission/>
-		<xacro:leg_gazebo/>
+		<xacro:leg_gazebo load_force_sensors="${load_force_sensors}"/>
 	</xacro:macro>
 </robot>

Commit message: [feature] Added the internal_wrench sensor
Conflicts:
	launch/empty_world.launch
	robots/hyl.urdf.xacro
	urdfs/leg/leg.gazebo.xacro

File: robots/hyl.urdf.xacro (robot description, xacro)
@@ -1,4 +1,6 @@
 <?xml version="1.0"?>
 <robot name="hyl" xmlns:xacro="http://www.ros.org/wiki/xacro">
+	<!-- This argument allows us to load joint sensors that measure the internal wrenches -->
+	<xacro:arg name="load_force_sensors" default="false"/>
 	<!-- The following included files set up definitions of parts of the robot body -->
 	<xacro:include filename="$(find hyl_description)/urdfs/common.xacro"/>
@@ -21,6 +23,6 @@
 	<xacro:hyl_support parent="world"/>
 	<!-- leg -->
-	<xacro:hyl_leg parent="base_link">
-		<origin xyz="0 0.025 0.85" rpy="0 0 0"/>
+	<xacro:hyl_leg parent="base_link" load_force_sensors="$(arg load_force_sensors)">
+		<origin xyz="0 0 0" rpy="0 0 0"/>
 	</xacro:hyl_leg>
 </robot>

File: urdfs/leg/leg.gazebo.xacro (robot description, xacro)
@@ -1,6 +1,45 @@
 <?xml version="1.0"?>
 <robot xmlns:xacro="http://www.ros.org/wiki/xacro">
-	<xacro:macro name="leg_gazebo">
-		<gazebo reference="lowerleg">
+	<xacro:macro name="leg_gazebo" params="load_force_sensors">
+		<gazebo reference="slider_joint">
+			<provideFeedback>true</provideFeedback>
+		</gazebo>
+		<xacro:if value="${load_force_sensors}">
+			<gazebo>
+				<plugin name="slider_sensor" filename="libgazebo_ros_ft_sensor.so">
+					<robotNamespace>/hyl/internal_wrench/</robotNamespace>
+					<updateRate>100.0</updateRate>
+					<topicName>slider_joint</topicName>
+					<jointName>slider_joint</jointName>
+				</plugin>
+			</gazebo>
+		</xacro:if>
+		<gazebo reference="kfe_joint">
+			<provideFeedback>true</provideFeedback>
+		</gazebo>
+		<xacro:if value="${load_force_sensors}">
+			<gazebo>
+				<plugin name="kfe_sensor" filename="libgazebo_ros_ft_sensor.so">
+					<robotNamespace>/hyl/internal_wrench/</robotNamespace>
+					<updateRate>100.0</updateRate>
+					<topicName>kfe_joint</topicName>
+					<jointName>kfe_joint</jointName>
+				</plugin>
+			</gazebo>
+		</xacro:if>
+		<gazebo reference="hfe_joint">
+			<provideFeedback>true</provideFeedback>
+		</gazebo>
+		<xacro:if value="${load_force_sensors}">
+			<gazebo>
+				<plugin name="hfe_sensor" filename="libgazebo_ros_ft_sensor.so">
+					<robotNamespace>/hyl/internal_wrench/</robotNamespace>
+					<updateRate>100.0</updateRate>
+					<topicName>hfe_joint</topicName>
+					<jointName>hfe_joint</jointName>
+				</plugin>
+			</gazebo>
+		</xacro:if>
+		<gazebo reference="foot">
 			<kp>1000000.0</kp>
 			<kd>100.0</kd>

File: urdfs/leg/leg.urdf.xacro (robot description, xacro)
@@ -6,5 +6,5 @@
 	<!-- ================================== Leg ================================== -->
 	<!-- The xacro macro xacro:hyl_leg contains: slider upper and lower leg -->
-	<xacro:macro name="hyl_leg" params="parent *origin">
+	<xacro:macro name="hyl_leg" params="parent *origin load_force_sensors">
 		<!-- Joints -->
 		<!-- Slider joint -->
@@ -155,5 +155,5 @@
 		<!-- Extensions -->
 		<xacro:leg_transmission/>
-		<xacro:leg_gazebo/>
+		<xacro:leg_gazebo load_force_sensors="${load_force_sensors}"/>
 	</xacro:macro>
 </robot>

Commit message: [stl] Added the STL files which are needed for bullet engine

File: robots/hyl.urdf.xacro (robot description, xacro)
@@ -3,4 +3,6 @@
 	<!-- This argument allows us to load joint sensors that measure the internal wrenches -->
 	<xacro:arg name="load_force_sensors" default="false"/>
+	<!-- This argument allows us to load STL mesh files instead of DAE ones -->
+	<xacro:arg name="stl" default="false"/>
 	<!-- The following included files set up definitions of parts of the robot body -->
 	<xacro:include filename="$(find hyl_description)/urdfs/common.xacro"/>
@@ -23,5 +25,7 @@
 	<xacro:hyl_support parent="world"/>
 	<!-- leg -->
-	<xacro:hyl_leg parent="base_link" load_force_sensors="$(arg load_force_sensors)">
+	<xacro:hyl_leg parent="base_link"
+		load_force_sensors="$(arg load_force_sensors)"
+		stl="$(arg stl)">
 		<origin xyz="0 0 0" rpy="0 0 0"/>
 	</xacro:hyl_leg>

File: urdfs/leg/leg.urdf.xacro (robot description, xacro)
@@ -6,5 +6,5 @@
 	<!-- ================================== Leg ================================== -->
 	<!-- The xacro macro xacro:hyl_leg contains: slider upper and lower leg -->
-	<xacro:macro name="hyl_leg" params="parent *origin load_force_sensors">
+	<xacro:macro name="hyl_leg" params="parent *origin load_force_sensors stl">
 		<!-- Joints -->
 		<!-- Slider joint -->
@@ -63,5 +63,10 @@
 				<origin xyz="0 0 0" rpy="-${PI/2} ${PI} 0"/>
 				<geometry>
-					<mesh filename="package://hyl_description/meshes/leg/trunk.dae" scale="1 1 1"/>
+					<xacro:if value="${stl}">
+						<mesh filename="package://hyl_description/meshes/leg/trunk.stl" scale="1 1 1"/>
+					</xacro:if>
+					<xacro:unless value="${stl}">
+						<mesh filename="package://hyl_description/meshes/leg/trunk.dae" scale="1 1 1"/>
+					</xacro:unless>
 				</geometry>
 				<material name="grey"/>
@@ -70,5 +75,10 @@
 				<origin xyz="0 0 0" rpy="-${PI/2} ${PI} 0"/>
 				<geometry>
-					<mesh filename="package://hyl_description/meshes/leg/trunk.dae" scale="1 1 1"/>
+					<xacro:if value="${stl}">
+						<mesh filename="package://hyl_description/meshes/leg/trunk.stl" scale="1 1 1"/>
+					</xacro:if>
+					<xacro:unless value="${stl}">
+						<mesh filename="package://hyl_description/meshes/leg/trunk.dae" scale="1 1 1"/>
+					</xacro:unless>
 				</geometry>
 			</collision>
@@ -85,12 +95,22 @@
 				<origin xyz="0 0 0" rpy="0 0 0"/>
 				<geometry>
-					<mesh filename="package://hyl_description/meshes/leg/hipassembly.dae" scale="1 1 1"/>
-				</geometry>
-				<material name="grey"/>
-			</visual>
-			<collision>
-				<origin xyz="0 0 0" rpy="0 0 0"/>
-				<geometry>
-					<mesh filename="package://hyl_description/meshes/leg/hipassembly.dae" scale="1 1 1"/>
+					<xacro:if value="${stl}">
+						<mesh filename="package://hyl_description/meshes/leg/hipassembly.stl" scale="1 1 1"/>
+					</xacro:if>
+					<xacro:unless value="${stl}">
+						<mesh filename="package://hyl_description/meshes/leg/hipassembly.dae" scale="1 1 1"/>
+					</xacro:unless>
+				</geometry>
+				<material name="grey"/>
+			</visual>
+			<collision>
+				<origin xyz="0 0 0" rpy="0 0 0"/>
+				<geometry>
+					<xacro:if value="${stl}">
+						<mesh filename="package://hyl_description/meshes/leg/hipassembly.stl" scale="1 1 1"/>
+					</xacro:if>
+					<xacro:unless value="${stl}">
+						<mesh filename="package://hyl_description/meshes/leg/hipassembly.dae" scale="1 1 1"/>
+					</xacro:unless>
 				</geometry>
 			</collision>
@@ -107,12 +127,22 @@
 				<origin xyz="0 0 0" rpy="0 0 0"/>
 				<geometry>
-					<mesh filename="package://hyl_description/meshes/leg/upperleg.dae" scale="1 1 1"/>
-				</geometry>
-				<material name="grey"/>
-			</visual>
-			<collision>
-				<origin xyz="0 0 0" rpy="0 0 0"/>
-				<geometry>
-					<mesh filename="package://hyl_description/meshes/leg/upperleg.dae" scale="1 1 1"/>
+					<xacro:if value="${stl}">
+						<mesh filename="package://hyl_description/meshes/leg/upperleg.stl" scale="1 1 1"/>
+					</xacro:if>
+					<xacro:unless value="${stl}">
+						<mesh filename="package://hyl_description/meshes/leg/upperleg.dae" scale="1 1 1"/>
+					</xacro:unless>
+				</geometry>
+				<material name="grey"/>
+			</visual>
+			<collision>
+				<origin xyz="0 0 0" rpy="0 0 0"/>
+				<geometry>
+					<xacro:if value="${stl}">
+						<mesh filename="package://hyl_description/meshes/leg/upperleg.stl" scale="1 1 1"/>
+					</xacro:if>
+					<xacro:unless value="${stl}">
+						<mesh filename="package://hyl_description/meshes/leg/upperleg.dae" scale="1 1 1"/>
+					</xacro:unless>
 				</geometry>
 			</collision>
@@ -128,11 +158,21 @@
 			<visual>
 				<geometry>
-					<mesh filename="package://hyl_description/meshes/leg/lowerleg.dae" scale="1 1 1"/>
-				</geometry>
-				<material name="grey"/>
-			</visual>
-			<collision>
-				<geometry>
-					<mesh filename="package://hyl_description/meshes/leg/lowerleg.dae" scale="1 1 1"/>
+					<xacro:if value="${stl}">
+						<mesh filename="package://hyl_description/meshes/leg/lowerleg.stl" scale="1 1 1"/>
+					</xacro:if>
+					<xacro:unless value="${stl}">
+						<mesh filename="package://hyl_description/meshes/leg/lowerleg.dae" scale="1 1 1"/>
+					</xacro:unless>
+				</geometry>
+				<material name="grey"/>
+			</visual>
+			<collision>
+				<geometry>
+					<xacro:if value="${stl}">
+						<mesh filename="package://hyl_description/meshes/leg/lowerleg.stl" scale="1 1 1"/>
+					</xacro:if>
+					<xacro:unless value="${stl}">
+						<mesh filename="package://hyl_description/meshes/leg/lowerleg.dae" scale="1 1 1"/>
+					</xacro:unless>
 				</geometry>
 			</collision>
