Commit message: Removed the haa joint definition

File: urdfs/leg/leg.transmission.xacro (robot description, xacro)
@@ -9,15 +9,4 @@
 			</joint>
 			<actuator name="slider_motor">
-				<hardwareInterface>EffortJointInterface</hardwareInterface>
-				<mechanicalReduction>1</mechanicalReduction>
-			</actuator>
-		</transmission>
-    	<!-- Upper leg -->
-		<transmission name="haa_trans">
-			<type>transmission_interface/SimpleTransmission</type>
-			<joint name="haa_joint">
-				<hardwareInterface>EffortJointInterface</hardwareInterface>
-			</joint>
-			<actuator name="haa_motor">
 				<hardwareInterface>EffortJointInterface</hardwareInterface>
 				<mechanicalReduction>1</mechanicalReduction>
