Commit message: Added a force sensor on the foot for debugging

File: urdfs/leg/leg.gazebo.xacro (robot description, xacro)
@@ -11,4 +11,21 @@
 			<minDepth>0.00</minDepth>
 		</gazebo>
+		<gazebo reference="foot">
+			<selfCollide>false</selfCollide>
+			<sensor type="contact" name="foot_contact_sensor">
+				<pose>0 0 0 0 0 0</pose>
+				<always_on>true</always_on>
+				<update_rate>100.0</update_rate>
+				<contact>
+					<collision>foot_collision</collision>
+				</contact>
+				<plugin name="foot_gazebo_ros_bumper_controller" filename="libgazebo_ros_bumper.so">
+					<alwaysOn>true</alwaysOn>
+					<updateRate>100.0</updateRate>
+					<bumperTopicName>/hyl/foot_force</bumperTopicName>
+					<frameName>world</frameName>
+				</plugin>
+			</sensor>
+		</gazebo>
 	</xacro:macro>
 </robot>

Commit message: Increased the size of the sphere in the foot in order to improved the contact simulation. Modified friction coeficient

File: urdfs/leg/leg.gazebo.xacro (robot description, xacro)
@@ -2,12 +2,12 @@
 <robot xmlns:xacro="http://www.ros.org/wiki/xacro">
 	<xacro:macro name="leg_gazebo">
-		<gazebo reference="lowerleg">
+		<gazebo reference="foot">
 			<kp>1000000.0</kp>
 			<kd>100.0</kd>
-			<mu1>1.5</mu1>
-			<mu2>1.5</mu2>
+			<mu1>0.8</mu1>
+			<mu2>0.8</mu2>
 			<fdir1>1 0 0</fdir1>
-			<maxVel>1.0</maxVel>
-			<minDepth>0.00</minDepth>
+			<maxVel>100.0</maxVel>
+			<minDepth>0.0</minDepth>
 		</gazebo>
 		<gazebo reference="foot">

File: urdfs/leg/leg.urdf.xacro (robot description, xacro)
@@ -145,5 +145,5 @@
 				<origin xyz="0 0 0" rpy="0 0 0"/>
 				<geometry>
-					<sphere radius="0.02175"/>
+					<sphere radius="0.02185"/>
 				</geometry>
 			</collision>

File: urdfs/support/support.urdf.xacro (robot description, xacro)
@@ -17,5 +17,5 @@
 			</inertial>
 			<collision>
-				<origin xyz="0 -0.025 -0.275" rpy="0 0 0" />
+				<origin xyz="0 -0.025 -0.27" rpy="0 0 0" />
 				<geometry>
 					<box size="0.12 0.045 1.15" />
@@ -23,5 +23,5 @@
 			</collision>
 			<visual>
-				<origin xyz="0 -0.025 -0.275" rpy="0 0 0" />
+				<origin xyz="0 -0.025 -0.27" rpy="0 0 0" />
 				<geometry>
 					<box size="0.12 0.045 1.15" />
