Commit message: Removed visual information of the foot

File: urdfs/leg/leg.urdf.xacro (robot description, xacro)
@@ -130,10 +130,4 @@
 				<inertia ixx="0.0" iyy="0.0" izz="0.0" ixy="0.0" ixz="0.0" iyz="0.0"/>
 			</inertial>
-			<visual>
-				<origin xyz="0.0 0.0 0.0" rpy="0.0 0.0 0.0"/>
-<!--				<geometry>
-					<sphere radius="0.021"/>
-				</geometry>-->
-			</visual>
 			<collision>
 				<origin xyz="0.0 0.0 0.0" rpy="0.0 0.0 0.0"/>

Commit message: Changed the name of the CAD to lowerleg and upperleg

File: urdfs/leg/leg.urdf.xacro (robot description, xacro)
@@ -98,5 +98,5 @@
 				<origin xyz="0 0 0" rpy="0 0 0"/>
 				<geometry>
-					<mesh filename="package://hyl_description/meshes/leg/upper.dae" scale="1 1 1"/>
+					<mesh filename="package://hyl_description/meshes/leg/upperleg.dae" scale="1 1 1"/>
 				</geometry>
 			</visual>
@@ -104,5 +104,5 @@
 				<origin xyz="0 0 0" rpy="0 0 0"/>
 				<geometry>
-					<mesh filename="package://hyl_description/meshes/leg/upper.dae" scale="1 1 1"/>
+					<mesh filename="package://hyl_description/meshes/leg/upperleg.dae" scale="1 1 1"/>
 				</geometry>
 			</collision>
@@ -118,5 +118,5 @@
 			<visual>
 				<geometry>
-					<mesh filename="package://hyl_description/meshes/leg/lower.dae" scale="1 1 1"/>
+					<mesh filename="package://hyl_description/meshes/leg/lowerleg.dae" scale="1 1 1"/>
 				</geometry>
 				<material name="white"/>
@@ -124,5 +124,5 @@
 			<collision>
 				<geometry>
-					<mesh filename="package://hyl_description/meshes/leg/lower.dae" scale="1 1 1"/>
+					<mesh filename="package://hyl_description/meshes/leg/lowerleg.dae" scale="1 1 1"/>
 				</geometry>
 			</collision>

Commit message: Added the hipassembly visual information

File: urdfs/leg/leg.urdf.xacro (robot description, xacro)
@@ -86,4 +86,16 @@
 						 ixy="${ixy_hipassembly}" ixz="${ixz_hipassembly}" iyz="${iyz_hipassembly}"/>
 			</inertial>
+			<visual>
+				<origin xyz="0 0 0" rpy="0 0 0"/>
+				<geometry>
+					<mesh filename="package://hyl_description/meshes/leg/hipassembly.dae" scale="1 1 1"/>
+				</geometry>
+			</visual>
+			<collision>
+				<origin xyz="0 0 0" rpy="0 0 0"/>
+				<geometry>
+					<mesh filename="package://hyl_description/meshes/leg/hipassembly.dae" scale="1 1 1"/>
+				</geometry>
+			</collision>
 		</link>
 		<!-- Upper leg link -->

Commit message: Remove friction and damping to the joints. We need to investigate these parameters with the real robot

File: urdfs/leg/leg.urdf.xacro (robot description, xacro)
@@ -15,5 +15,5 @@
 			<limit effort="100000.0" velocity="100.0" lower="-0.60" upper="0.5"/>
 			<axis xyz="0 0 1"/>
-			<dynamics damping="0.1" friction="0" />
+			<dynamics damping="0" friction="0" />
 		</joint>
 		<!-- Hip assembly joint -->
@@ -30,5 +30,5 @@
 			<limit effort="200.0" velocity="1000.0" lower="${-PI/2}" upper="${PI/6}"/>
 			<axis xyz="0 0 1"/>
-			<dynamics damping="0.1" friction="0" />
+			<dynamics damping="0" friction="0" />
 			<safety_controller k_position="100" k_velocity="100" soft_lower_limit="-10" soft_upper_limit="12.45" />
 		</joint>
@@ -41,5 +41,5 @@
 				   upper="${14*PI/36}"/>
 			<axis xyz="0 0 1"/>
-			<dynamics damping="0.1" friction="0" />
+			<dynamics damping="0" friction="0" />
 			<safety_controller k_position="100" k_velocity="100" soft_lower_limit="-10" soft_upper_limit="12.45" />
 		</joint>
@@ -52,5 +52,5 @@
 				   upper="${-2*PI/18}"/>
 			<axis xyz="0 0 1"/>
-			<dynamics damping="0.1" friction="0" />
+			<dynamics damping="0" friction="0" />
 			<safety_controller k_position="100" k_velocity="100" soft_lower_limit="-10" soft_upper_limit="12.45" />
 		</joint>

Commit message: Added the right values for the maximum effort and velocity of every joint

File: urdfs/leg/leg.urdf.xacro (robot description, xacro)
@@ -28,5 +28,5 @@
 			<parent link="assembly"/>
 			<child  link="hipassembly"/>
-			<limit effort="200.0" velocity="1000.0" lower="${-PI/2}" upper="${PI/6}"/>
+			<limit effort="150.0" velocity="12.0" lower="${-PI/2}" upper="${PI/6}"/>
 			<axis xyz="0 0 1"/>
 			<dynamics damping="0" friction="0" />
@@ -38,5 +38,5 @@
 			<parent link="hipassembly"/>
 			<child  link="upperleg"/>
-			<limit effort="200.0" velocity="1.0" lower="${-10*PI/36}"
+			<limit effort="150.0" velocity="12.0" lower="${-10*PI/36}"
 				   upper="${14*PI/36}"/>
 			<axis xyz="0 0 1"/>
@@ -49,5 +49,5 @@
 			<parent link="upperleg"/>
 			<child  link="lowerleg"/>
-			<limit effort="200.0" velocity="1.0" lower="${-14*PI/18}"
+			<limit effort="150.0" velocity="12.0" lower="${-14*PI/18}"
 				   upper="${-2*PI/18}"/>
 			<axis xyz="0 0 1"/>

Commit message: Removed the assembly link that is useless

File: urdfs/leg/leg.urdf.xacro (robot description, xacro)
@@ -18,13 +18,7 @@
 		</joint>
 		<!-- Hip assembly joint -->
-		<joint name="assembly_joint" type="fixed">
+		<joint name="haa_joint" type="revolute">
 			<origin xyz="0 ${d_lr/2} 0" rpy="0 ${PI/2} ${PI}"/>
 			<parent link="slider"/>
-			<child  link="assembly"/>
-		</joint>
-		<!-- Virtual hip joint assembly -->
-		<joint name="haa_joint" type="revolute">
-			<origin xyz="0 0 0" rpy="0 0 0"/>
-			<parent link="assembly"/>
 			<child  link="hipassembly"/>
 			<limit effort="150.0" velocity="12.0" lower="${-PI/2}" upper="${PI/6}"/>
@@ -64,12 +58,4 @@
 		<!-- Slider link -->
 		<link name="slider">
-			<inertial>
-				<origin xyz="0 0 0"/>
-				<mass value="0.01"/>
-				<inertia ixx="0.01" iyy="0.01" izz="0.01" ixy="0.0" ixz="0.0" iyz="0.0"/>
-			</inertial>
-		</link>
-		<!-- Leg assembly link -->
-		<link name="assembly">
 			<inertial>
 				<origin xyz="0 0 0"/>

Commit message: Defined the haa_joint as a fixed joint

File: urdfs/leg/leg.urdf.xacro (robot description, xacro)
@@ -18,5 +18,5 @@
 		</joint>
 		<!-- Hip assembly joint -->
-		<joint name="haa_joint" type="revolute">
+		<joint name="haa_joint" type="fixed">
 			<origin xyz="0 ${d_lr/2} 0" rpy="0 ${PI/2} ${PI}"/>
 			<parent link="slider"/>

Commit message: Changed the name of the slider link to trunk because is more general to floating-base platforms

File: urdfs/leg/leg.urdf.xacro (robot description, xacro)
@@ -12,5 +12,5 @@
 			<insert_block name="origin"/>
 			<parent link="${parent}"/>
-			<child  link="slider"/>
+			<child  link="trunk"/>
 			<limit effort="100000.0" velocity="100.0" lower="-0.60" upper="0.5"/>
 			<axis xyz="0 0 1"/>
@@ -20,5 +20,5 @@
 		<joint name="haa_joint" type="fixed">
 			<origin xyz="0 ${d_lr/2} 0" rpy="0 ${PI/2} ${PI}"/>
-			<parent link="slider"/>
+			<parent link="trunk"/>
 			<child  link="hipassembly"/>
 			<limit effort="150.0" velocity="12.0" lower="${-PI/2}" upper="${PI/6}"/>
@@ -56,6 +56,6 @@
 		</joint>
 		<!-- Links -->
-		<!-- Slider link -->
-		<link name="slider">
+		<!-- Trunk link -->
+		<link name="trunk">
 			<inertial>
 				<origin xyz="0 0 0"/>

Commit message: Changed the name of the slider link to trunk because is more general to floating-base platforms

File: urdfs/leg/leg.urdf.xacro (robot description, xacro)
@@ -12,5 +12,5 @@
 			<insert_block name="origin"/>
 			<parent link="${parent}"/>
-			<child  link="slider"/>
+			<child  link="trunk"/>
 			<limit effort="100000.0" velocity="100.0" lower="-0.60" upper="0.5"/>
 			<axis xyz="0 0 1"/>
@@ -20,5 +20,5 @@
 		<joint name="haa_joint" type="revolute">
 			<origin xyz="0 ${d_lr/2} 0" rpy="0 ${PI/2} ${PI}"/>
-			<parent link="slider"/>
+			<parent link="trunk"/>
 			<child  link="hipassembly"/>
 			<limit effort="150.0" velocity="12.0" lower="${-PI/2}" upper="${PI/6}"/>
@@ -56,6 +56,6 @@
 		</joint>
 		<!-- Links -->
-		<!-- Slider link -->
-		<link name="slider">
+		<!-- Trunk link -->
+		<link name="trunk">
 			<inertial>
 				<origin xyz="0 0 0"/>

Commit message: Added visual and inertial properties of trunk

File: urdfs/leg/leg.urdf.xacro (robot description, xacro)
@@ -59,8 +59,21 @@
 		<link name="trunk">
 			<inertial>
-				<origin xyz="0 0 0"/>
-				<mass value="0.01"/>
-				<inertia ixx="0.01" iyy="0.01" izz="0.01" ixy="0.0" ixz="0.0" iyz="0.0"/>
+				<origin xyz="${xcom_trunk} ${ycom_trunk} ${zcom_trunk}"/>
+				<mass value="${m_trunk}"/>
+				<inertia ixx="${ixx_trunk}" iyy="${iyy_trunk}" izz="${izz_trunk}"
+						 ixy="${ixy_trunk}" ixz="${ixz_trunk}" iyz="${iyz_trunk}"/>
 			</inertial>
+			<visual>
+				<origin xyz="0 0 0" rpy="-${PI/2} ${PI} 0"/>
+				<geometry>
+					<mesh filename="package://hyl_description/meshes/leg/trunk.dae" scale="1 1 1"/>
+				</geometry>
+			</visual>
+			<collision>
+				<origin xyz="0 0 0" rpy="-${PI/2} ${PI} 0"/>
+				<geometry>
+					<mesh filename="package://hyl_description/meshes/leg/trunk.dae" scale="1 1 1"/>
+				</geometry>
+			</collision>
 		</link>
 		<!-- Hip assembly link -->

Commit message: Defined the HAA as a non-fixed joint because the HyL SL is setup like this. Otherwise we cannot visualize in rviz because defined joint are inconsistent

File: urdfs/leg/leg.urdf.xacro (robot description, xacro)
@@ -18,5 +18,5 @@
 		</joint>
 		<!-- Hip assembly joint -->
-		<joint name="haa_joint" type="fixed">
+		<joint name="haa_joint" type="revolute">
 			<origin xyz="0 ${d_lr/2} 0" rpy="0 ${PI/2} ${PI}"/>
 			<parent link="trunk"/>

Commit message: Defined the maximum effort in the slider as 0 because isn't actuated this joint

File: urdfs/leg/leg.urdf.xacro (robot description, xacro)
@@ -13,5 +13,5 @@
 			<parent link="${parent}"/>
 			<child  link="trunk"/>
-			<limit effort="100000.0" velocity="100.0" lower="-0.60" upper="0.5"/>
+			<limit effort="0.0" velocity="100.0" lower="-0.60" upper="0.5"/>
 			<axis xyz="0 0 1"/>
 			<dynamics damping="0" friction="0" />
