Commit message: Removed a coupled comment lines

File: urdfs/support/support.urdf.xacro (robot description, xacro)
@@ -20,5 +20,4 @@
 				<geometry>
 					<box size="0.12 0.045 1.15" />
-<!--					<mesh filename="package://hyq_description/meshes/trunk/trunk_frame.dae" scale="1 1 1"/>-->
 				</geometry>
 			</collision>
@@ -27,5 +26,4 @@
 				<geometry>
 					<box size="0.12 0.045 1.15" />
-<!--					<mesh filename="package://hyq_description/meshes/trunk/trunk_frame.dae" scale="1 1 1"/>-->
 				</geometry>
 			</visual>

Commit message: Changed the color of the support

File: urdfs/support/support.urdf.xacro (robot description, xacro)
@@ -27,4 +27,7 @@
 					<box size="0.12 0.045 1.15" />
 				</geometry>
+				<material name="blue">
+					<color rgba="0.2 0.2 0.2 1"/>
+				</material>
 			</visual>
 		</link>
