Commit message: Removed the initial position definition that is useless

File: urdfs/common.xacro (robot description, xacro)
@@ -6,7 +6,4 @@
 	<property name="d_tbb" value="0.0825"/>
 	<property name="d_p1p2" value="0.35"/>
-	<!-- Initial joint positions -->
-	<property name="hfe_pos0" value="0"/>
-	<property name="kfe_pos0" value="0"/>
 	<!-- Inertial values -->
 	<!-- Trunk with hydraulic system -->

File: urdfs/leg/leg.urdf.xacro (robot description, xacro)
@@ -35,8 +35,8 @@
 		<!-- Upper leg joint -->
 		<joint name="hfe_joint" type="revolute">
-			<origin xyz="${d_tbb} 0.0 0.0" rpy="${reflect_upper*PI/2} ${-1*hfe_pos0} 0.0"/>
+			<origin xyz="${d_tbb} 0.0 0.0" rpy="${reflect_upper*PI/2} 0 0"/>
 			<parent link="hipassembly"/>
 			<child  link="upperleg"/>
-			<limit effort="200.0" velocity="1.0" lower="${-(1+reflect_front)*5*PI/36-(1-reflect_front)*7*PI/36-reflect_front*hfe_pos0}" upper="${(1-reflect_front)*5*PI/36+(1+reflect_front)*7*PI/36-reflect_front*hfe_pos0}"/>
+			<limit effort="200.0" velocity="1.0" lower="${-(1+reflect_front)*5*PI/36-(1-reflect_front)*7*PI/36}" upper="${(1-reflect_front)*5*PI/36+(1+reflect_front)*7*PI/36}"/>
 			<axis xyz="0 0 1"/>
 			<dynamics damping="0.1" friction="0" />
@@ -45,8 +45,8 @@
 		<!-- Lower leg joint -->
 		<joint name="kfe_joint" type="revolute">
-			<origin xyz="${d_p1p2} 0.0 0.0" rpy="0.0 0.0 ${reflect_front*kfe_pos0}"/>
+			<origin xyz="${d_p1p2} 0.0 0.0" rpy="0 0 0"/>
 			<parent link="upperleg"/>
 			<child  link="lowerleg"/>
-			<limit effort="200.0" velocity="1.0" lower="${-(1+reflect_front)*7*PI/18+(1-reflect_front)*PI/18-reflect_front*kfe_pos0}" upper="${(1-reflect_front)*7*PI/18-(1+reflect_front)*PI/18-reflect_front*kfe_pos0}"/>
+			<limit effort="200.0" velocity="1.0" lower="${-(1+reflect_front)*7*PI/18+(1-reflect_front)*PI/18}" upper="${(1-reflect_front)*7*PI/18-(1+reflect_front)*PI/18}"/>
 			<axis xyz="0 0 1"/>
 			<dynamics damping="0.1" friction="0" />

Commit message: Changed the inertial parameter according to Marco' values (robcogen)

File: urdfs/common.xacro (robot description, xacro)
@@ -15,19 +15,36 @@
 	<property name="ixz_trunk" value="-0.06"/>
 	<property name="iyz_trunk" value="-0.03"/>
+	<!-- Hip assembly leg -->
+	<property name="xcom_hipassembly" value="0.03951"/>
+	<property name="ycom_hipassembly" value="0.00023"/>
+	<property name="zcom_hipassembly" value="0.16045"/>
+	<property name="m_hipassembly" value="2.7754"/>
+	<property name="ixx_hipassembly" value="0.122710"/>
+	<property name="iyy_hipassembly" value="0.130957"/>
+	<property name="izz_hipassembly" value="0.009731"/>
+	<property name="ixy_hipassembly" value="0.000022"/>
+	<property name="ixz_hipassembly" value="0.018692"/>
+	<property name="iyz_hipassembly" value="0.000007"/>
 	<!-- Upper leg -->
-	<property name="m_upper" value="2.16"/>
-	<property name="ixx_upper" value="0.004785"/>
-	<property name="iyy_upper" value="0.076166"/>
-	<property name="izz_upper" value="0.078576"/>
-	<property name="ixy_upper" value="0.0071588"/>
-	<property name="ixz_upper" value="0.0"/>
-	<property name="iyz_upper" value="0.0"/>
+	<property name="xcom_upperleg" value="0.14925"/>
+	<property name="ycom_upperleg" value="-0.02996"/>
+	<property name="zcom_upperleg" value="-0.00005"/>
+	<property name="m_upperleg" value="2.06218"/>
+	<property name="ixx_upperleg" value="0.00464"/>
+	<property name="iyy_upperleg" value="0.07216"/>
+	<property name="izz_upperleg" value="0.07463"/>
+	<property name="ixy_upperleg" value="-0.00718"/>
+	<property name="ixz_upperleg" value="-0.00001"/>
+	<property name="iyz_upperleg" value="-0.00001"/>
 	<!-- Lower leg -->
-	<property name="m_lower" value="1.8717"/>
-	<property name="ixx_lower" value="9.0E-4"/>
-	<property name="iyy_lower" value="0.0777"/>
-	<property name="izz_lower" value="0.0775"/>
-	<property name="ixy_lower" value="-0.0"/>
-	<property name="ixz_lower" value="-0.0"/>
-	<property name="iyz_lower" value="0.0"/>
+	<property name="xcom_lowerleg" value="0.12185"/>
+	<property name="ycom_lowerleg" value="0.00058"/>
+	<property name="zcom_lowerleg" value="-0.00012"/>
+	<property name="m_lowerleg" value="0.80669"/>
+	<property name="ixx_lowerleg" value="0.00042"/>
+	<property name="iyy_lowerleg" value="0.02202"/>
+	<property name="izz_lowerleg" value="0.02183"/>
+	<property name="ixy_lowerleg" value="0.0"/>
+	<property name="ixz_lowerleg" value="0.0"/>
+	<property name="iyz_lowerleg" value="0.0"/>
 </robot>

File: urdfs/leg/leg.urdf.xacro (robot description, xacro)
@@ -35,8 +35,9 @@
 		<!-- Upper leg joint -->
 		<joint name="hfe_joint" type="revolute">
-			<origin xyz="${d_tbb} 0.0 0.0" rpy="${reflect_upper*PI/2} 0 0"/>
+			<origin xyz="${d_tbb} 0 0" rpy="${reflect_upper*PI/2} 0 0"/>
 			<parent link="hipassembly"/>
 			<child  link="upperleg"/>
-			<limit effort="200.0" velocity="1.0" lower="${-(1+reflect_front)*5*PI/36-(1-reflect_front)*7*PI/36}" upper="${(1-reflect_front)*5*PI/36+(1+reflect_front)*7*PI/36}"/>
+			<limit effort="200.0" velocity="1.0" lower="${-(1+reflect_front)*5*PI/36-(1-reflect_front)*7*PI/36}"
+				   upper="${(1-reflect_front)*5*PI/36+(1+reflect_front)*7*PI/36}"/>
 			<axis xyz="0 0 1"/>
 			<dynamics damping="0.1" friction="0" />
@@ -45,8 +46,9 @@
 		<!-- Lower leg joint -->
 		<joint name="kfe_joint" type="revolute">
-			<origin xyz="${d_p1p2} 0.0 0.0" rpy="0 0 0"/>
+			<origin xyz="${d_p1p2} 0 0" rpy="0 0 0"/>
 			<parent link="upperleg"/>
 			<child  link="lowerleg"/>
-			<limit effort="200.0" velocity="1.0" lower="${-(1+reflect_front)*7*PI/18+(1-reflect_front)*PI/18}" upper="${(1-reflect_front)*7*PI/18-(1+reflect_front)*PI/18}"/>
+			<limit effort="200.0" velocity="1.0" lower="${-(1+reflect_front)*7*PI/18+(1-reflect_front)*PI/18}"
+				   upper="${(1-reflect_front)*7*PI/18-(1+reflect_front)*PI/18}"/>
 			<axis xyz="0 0 1"/>
 			<dynamics damping="0.1" friction="0" />
@@ -55,5 +57,5 @@
 		<!-- Foot joint -->
 		<joint name="foot_joint" type="fixed">
-			<origin xyz="0.34 0.0 0.0" rpy="${PI/2} 0.0 ${-PI/2}"/>
+			<origin xyz="0.34 0 0" rpy="${PI/2} 0 ${-PI/2}"/>
 			<parent link="lowerleg"/>
 			<child  link="foot"/>
@@ -63,5 +65,5 @@
 		<link name="slider">
 			<inertial>
-				<origin xyz="0.0 0.0 0.0"/>
+				<origin xyz="0 0 0"/>
 				<mass value="0.01"/>
 				<inertia ixx="0.01" iyy="0.01" izz="0.01" ixy="0.0" ixz="0.0" iyz="0.0"/>
@@ -71,5 +73,5 @@
 		<link name="assembly">
 			<inertial>
-				<origin xyz="0.0 0.0 0.0"/>
+				<origin xyz="0 0 0"/>
 				<mass value="0.01"/>
 				<inertia ixx="0.01" iyy="0.01" izz="0.01" ixy="0.0" ixz="0.0" iyz="0.0"/>
@@ -79,7 +81,8 @@
 		<link name="hipassembly">
 			<inertial>
-				<origin xyz="0.0 0.0 0.0"/>
-				<mass value="0.01"/>
-				<inertia ixx="0.01" iyy="0.01" izz="0.01" ixy="0.0" ixz="0.0" iyz="0.0"/>
+				<origin xyz="${xcom_hipassembly} ${ycom_hipassembly} ${zcom_hipassembly}"/>
+				<mass value="${m_hipassembly}"/>
+				<inertia ixx="${ixx_hipassembly}" iyy="${iyy_hipassembly}" izz="${izz_hipassembly}"
+						 ixy="${ixy_hipassembly}" ixz="${ixz_hipassembly}" iyz="${iyz_hipassembly}"/>
 			</inertial>
 		</link>
@@ -87,10 +90,11 @@
 		<link name="upperleg">
 			<inertial>
-				<origin xyz="0.14796 ${reflect_upper*0.02958} 0.0"/>
-				<mass value="${m_upper}"/>
-				<inertia ixx="${ixx_upper}" iyy="${iyy_upper}" izz="${izz_upper}" ixy="${ixy_upper}" ixz="${ixz_upper}" iyz="${iyz_upper}"/>
+				<origin xyz="${xcom_upperleg} ${reflect_upper*ycom_upperleg} ${zcom_upperleg}"/>
+				<mass value="${m_upperleg}"/>
+				<inertia ixx="${ixx_upperleg}" iyy="${iyy_upperleg}" izz="${izz_upperleg}"
+						 ixy="${ixy_upperleg}" ixz="${ixz_upperleg}" iyz="${iyz_upperleg}"/>
 			</inertial>
 			<visual>
-				<origin xyz="0.0 0.0 0.0" rpy="${(1-reflect_front)*PI/2} 0.0 0.0"/>
+				<origin xyz="0 0 0" rpy="${(1-reflect_front)*PI/2} 0 0"/>
 				<geometry>
 					<mesh filename="package://hyl_description/meshes/leg/upper.dae" scale="1 1 1"/>
@@ -98,5 +102,5 @@
 			</visual>
 			<collision>
-				<origin xyz="0.0 0.0 0.0" rpy="${(1-reflect_front)*PI/2} 0.0 0.0"/>
+				<origin xyz="0 0 0" rpy="${(1-reflect_front)*PI/2} 0 0"/>
 				<geometry>
 					<mesh filename="package://hyl_description/meshes/leg/upper.dae" scale="1 1 1"/>
@@ -107,7 +111,8 @@
 		<link name="lowerleg">
 			<inertial>
-				<origin xyz=" 0.17830  0.00030 -0.00010"/>
-				<mass value="${m_lower}"/>
-				<inertia ixx="${ixx_lower}" iyy="${iyy_lower}" izz="${izz_lower}" ixy="${ixy_lower}" ixz="${ixz_lower}" iyz="${iyz_lower}"/>
+				<origin xyz="${xcom_lowerleg} ${ycom_lowerleg} ${zcom_lowerleg}"/>
+				<mass value="${m_lowerleg}"/>
+				<inertia ixx="${ixx_lowerleg}" iyy="${iyy_lowerleg}" izz="${izz_lowerleg}"
+						 ixy="${ixy_lowerleg}" ixz="${ixz_lowerleg}" iyz="${iyz_lowerleg}"/>
 			</inertial>
 			<visual>
@@ -126,10 +131,10 @@
 		<link name="foot">
 			<inertial>
-				<origin xyz="0.0 0.0 0.0"/>
+				<origin xyz="0 0 0"/>
 				<mass value="0.01"/>
 				<inertia ixx="0.0" iyy="0.0" izz="0.0" ixy="0.0" ixz="0.0" iyz="0.0"/>
 			</inertial>
 			<collision>
-				<origin xyz="0.0 0.0 0.0" rpy="0.0 0.0 0.0"/>
+				<origin xyz="0 0 0" rpy="0 0 0"/>
 				<geometry>
 					<sphere radius="0.02175"/>

Commit message: Added visual and inertial properties of trunk

File: urdfs/common.xacro (robot description, xacro)
@@ -3,8 +3,19 @@
 	<property name="PI" value="3.1415926535897931"/>
 	<!-- standard distances -->
-	<property name="d_lr" value="0.25"/>
+	<property name="d_lr" value="0.26"/>
 	<property name="d_tbb" value="0.0825"/>
 	<property name="d_p1p2" value="0.35"/>
 	<!-- Inertial values -->
+	<!-- Trunk -->
+	<property name="xcom_trunk" value="-0.06532"/>
+	<property name="ycom_trunk" value="0.04079"/>
+	<property name="zcom_trunk" value="-0.01136"/>
+	<property name="m_trunk" value="2.5893"/>
+	<property name="ixx_trunk" value="0.012727"/>
+	<property name="iyy_trunk" value="0.041992"/>
+	<property name="izz_trunk" value="0.047339"/>
+	<property name="ixy_trunk" value="0.008496"/>
+	<property name="ixz_trunk" value="-0.0000107"/>
+	<property name="iyz_trunk" value="0.00000331"/>
 	<!-- Hip assembly leg -->
 	<property name="xcom_hipassembly" value="0.03951"/>

File: urdfs/leg/leg.urdf.xacro (robot description, xacro)
@@ -59,8 +59,21 @@
 		<link name="trunk">
 			<inertial>
-				<origin xyz="0 0 0"/>
-				<mass value="0.01"/>
-				<inertia ixx="0.01" iyy="0.01" izz="0.01" ixy="0.0" ixz="0.0" iyz="0.0"/>
+				<origin xyz="${xcom_trunk} ${ycom_trunk} ${zcom_trunk}"/>
+				<mass value="${m_trunk}"/>
+				<inertia ixx="${ixx_trunk}" iyy="${iyy_trunk}" izz="${izz_trunk}"
+						 ixy="${ixy_trunk}" ixz="${ixz_trunk}" iyz="${iyz_trunk}"/>
 			</inertial>
+			<visual>
+				<origin xyz="0 0 0" rpy="-${PI/2} ${PI} 0"/>
+				<geometry>
+					<mesh filename="package://hyl_description/meshes/leg/trunk.dae" scale="1 1 1"/>
+				</geometry>
+			</visual>
+			<collision>
+				<origin xyz="0 0 0" rpy="-${PI/2} ${PI} 0"/>
+				<geometry>
+					<mesh filename="package://hyl_description/meshes/leg/trunk.dae" scale="1 1 1"/>
+				</geometry>
+			</collision>
 		</link>
 		<!-- Hip assembly link -->

Commit message: Removed extra information that is not required for a fixed HAA joint

File: urdfs/common.xacro (robot description, xacro)
@@ -19,14 +19,4 @@
 	<property name="iyz_trunk" value="0.003392"/>
 	<!-- Hip assembly leg -->
-<!--	<property name="xcom_hipassembly" value="0.03951"/>
-	<property name="ycom_hipassembly" value="0.00023"/>
-	<property name="zcom_hipassembly" value="0.16045"/>
-	<property name="m_hipassembly" value="2.7754"/>
-	<property name="ixx_hipassembly" value="0.122710"/>
-	<property name="iyy_hipassembly" value="0.130957"/>
-	<property name="izz_hipassembly" value="0.009731"/>
-	<property name="ixy_hipassembly" value="0.000022"/>
-	<property name="ixz_hipassembly" value="0.018692"/>
-	<property name="iyz_hipassembly" value="0.000007"/>-->
 	<property name="xcom_hipassembly" value="0.0"/>
 	<property name="ycom_hipassembly" value="0.0"/>

File: urdfs/leg/leg.urdf.xacro (robot description, xacro)
@@ -18,12 +18,8 @@
 		</joint>
 		<!-- Hip assembly joint -->
-		<joint name="haa_joint" type="revolute">
+		<joint name="haa_joint" type="fixed">
 			<origin xyz="0 ${d_lr/2} 0" rpy="0 ${PI/2} ${PI}"/>
 			<parent link="trunk"/>
 			<child  link="hipassembly"/>
-			<limit effort="150.0" velocity="12.0" lower="${-PI/2}" upper="${PI/6}"/>
-			<axis xyz="0 0 1"/>
-			<dynamics damping="0" friction="0" />
-			<safety_controller k_position="100" k_velocity="100" soft_lower_limit="-10" soft_upper_limit="12.45" />
 		</joint>
 		<!-- Upper leg joint -->

Commit message: Propagate the values of the HyQV1LegV2_StandardDefinitions_v3.pdf to HyL

File: urdfs/common.xacro (robot description, xacro)
@@ -4,6 +4,7 @@
 	<!-- standard distances -->
 	<property name="d_lr" value="0.26"/>
-	<property name="d_tbb" value="0.0825"/>
+	<property name="d_p0p1" value="0.08"/>
 	<property name="d_p1p2" value="0.35"/>
+	<property name="d_p2p3" value="0.341"/>
 	<!-- Inertial values -->
 	<!-- Trunk -->

File: urdfs/leg/leg.urdf.xacro (robot description, xacro)
@@ -29,5 +29,5 @@
 		<!-- Upper leg joint -->
 		<joint name="hfe_joint" type="revolute">
-			<origin xyz="${d_tbb} 0 0" rpy="${PI/2} 0 0"/>
+			<origin xyz="${d_p0p1} 0 0" rpy="${PI/2} 0 0"/>
 			<parent link="hipassembly"/>
 			<child  link="upperleg"/>
@@ -51,5 +51,5 @@
 		<!-- Foot joint -->
 		<joint name="foot_joint" type="fixed">
-			<origin xyz="0.34 0 0" rpy="${PI/2} 0 ${-PI/2}"/>
+			<origin xyz="${d_p2p3} 0 0" rpy="${PI/2} 0 ${-PI/2}"/>
 			<parent link="lowerleg"/>
 			<child  link="foot"/>

Commit message: Propagate the values of the HyQV1LegV2_StandardDefinitions_v3.pdf to HyL

File: urdfs/common.xacro (robot description, xacro)
@@ -4,6 +4,7 @@
 	<!-- standard distances -->
 	<property name="d_lr" value="0.26"/>
-	<property name="d_tbb" value="0.0825"/>
+	<property name="d_p0p1" value="0.08"/>
 	<property name="d_p1p2" value="0.35"/>
+	<property name="d_p2p3" value="0.341"/>
 	<!-- Inertial values -->
 	<!-- Trunk -->

File: urdfs/leg/leg.urdf.xacro (robot description, xacro)
@@ -25,5 +25,5 @@
 		<!-- Upper leg joint -->
 		<joint name="hfe_joint" type="revolute">
-			<origin xyz="${d_tbb} 0 0" rpy="${PI/2} 0 0"/>
+			<origin xyz="${d_p0p1} 0 0" rpy="${PI/2} 0 0"/>
 			<parent link="hipassembly"/>
 			<child  link="upperleg"/>
@@ -47,5 +47,5 @@
 		<!-- Foot joint -->
 		<joint name="foot_joint" type="fixed">
-			<origin xyz="0.34 0 0" rpy="${PI/2} 0 ${-PI/2}"/>
+			<origin xyz="${d_p2p3} 0 0" rpy="${PI/2} 0 ${-PI/2}"/>
 			<parent link="lowerleg"/>
 			<child  link="foot"/>

Commit message: Fix tags for xacro in kinetic

File: urdfs/common.xacro (robot description, xacro)
@@ -1,54 +1,54 @@
 <?xml version="1.0"?>
 <robot>
-	<property name="PI" value="3.1415926535897931"/>
+	<xacro:property name="PI" value="3.1415926535897931"/>
 	<!-- standard distances -->
-	<property name="d_lr" value="0.26"/>
-	<property name="d_p0p1" value="0.08"/>
-	<property name="d_p1p2" value="0.35"/>
-	<property name="d_p2p3" value="0.341"/>
+	<xacro:property name="d_lr" value="0.26"/>
+	<xacro:property name="d_p0p1" value="0.08"/>
+	<xacro:property name="d_p1p2" value="0.35"/>
+	<xacro:property name="d_p2p3" value="0.341"/>
 	<!-- Inertial values -->
 	<!-- Trunk -->
-	<property name="xcom_trunk" value="-0.08315"/>
-	<property name="ycom_trunk" value="0.06849"/>
-	<property name="zcom_trunk" value="-0.00654"/>
-	<property name="m_trunk" value="7.982"/>
-	<property name="ixx_trunk" value="0.037131"/>
-	<property name="iyy_trunk" value="0.087473"/>
-	<property name="izz_trunk" value="0.112496"/>
-	<property name="ixy_trunk" value="0.028543"/>
-	<property name="ixz_trunk" value="-0.00097"/>
-	<property name="iyz_trunk" value="0.003392"/>
+	<xacro:property name="xcom_trunk" value="-0.08315"/>
+	<xacro:property name="ycom_trunk" value="0.06849"/>
+	<xacro:property name="zcom_trunk" value="-0.00654"/>
+	<xacro:property name="m_trunk" value="7.982"/>
+	<xacro:property name="ixx_trunk" value="0.037131"/>
+	<xacro:property name="iyy_trunk" value="0.087473"/>
+	<xacro:property name="izz_trunk" value="0.112496"/>
+	<xacro:property name="ixy_trunk" value="0.028543"/>
+	<xacro:property name="ixz_trunk" value="-0.00097"/>
+	<xacro:property name="iyz_trunk" value="0.003392"/>
 	<!-- Hip assembly leg -->
-	<property name="xcom_hipassembly" value="0.0"/>
-	<property name="ycom_hipassembly" value="0.0"/>
-	<property name="zcom_hipassembly" value="0.0"/>
-	<property name="m_hipassembly" value="0.001"/>
-	<property name="ixx_hipassembly" value="0.001"/>
-	<property name="iyy_hipassembly" value="0.001"/>
-	<property name="izz_hipassembly" value="0.001"/>
-	<property name="ixy_hipassembly" value="0.0"/>
-	<property name="ixz_hipassembly" value="0.0"/>
-	<property name="iyz_hipassembly" value="0.0"/>
+	<xacro:property name="xcom_hipassembly" value="0.0"/>
+	<xacro:property name="ycom_hipassembly" value="0.0"/>
+	<xacro:property name="zcom_hipassembly" value="0.0"/>
+	<xacro:property name="m_hipassembly" value="0.001"/>
+	<xacro:property name="ixx_hipassembly" value="0.001"/>
+	<xacro:property name="iyy_hipassembly" value="0.001"/>
+	<xacro:property name="izz_hipassembly" value="0.001"/>
+	<xacro:property name="ixy_hipassembly" value="0.0"/>
+	<xacro:property name="ixz_hipassembly" value="0.0"/>
+	<xacro:property name="iyz_hipassembly" value="0.0"/>
 	<!-- Upper leg -->
-	<property name="xcom_upperleg" value="0.14925"/>
-	<property name="ycom_upperleg" value="-0.02996"/>
-	<property name="zcom_upperleg" value="-0.00005"/>
-	<property name="m_upperleg" value="2.06218"/>
-	<property name="ixx_upperleg" value="0.00464"/>
-	<property name="iyy_upperleg" value="0.07216"/>
-	<property name="izz_upperleg" value="0.07463"/>
-	<property name="ixy_upperleg" value="-0.00718"/>
-	<property name="ixz_upperleg" value="-0.00001"/>
-	<property name="iyz_upperleg" value="-0.00001"/>
+	<xacro:property name="xcom_upperleg" value="0.14925"/>
+	<xacro:property name="ycom_upperleg" value="-0.02996"/>
+	<xacro:property name="zcom_upperleg" value="-0.00005"/>
+	<xacro:property name="m_upperleg" value="2.06218"/>
+	<xacro:property name="ixx_upperleg" value="0.00464"/>
+	<xacro:property name="iyy_upperleg" value="0.07216"/>
+	<xacro:property name="izz_upperleg" value="0.07463"/>
+	<xacro:property name="ixy_upperleg" value="-0.00718"/>
+	<xacro:property name="ixz_upperleg" value="-0.00001"/>
+	<xacro:property name="iyz_upperleg" value="-0.00001"/>
 	<!-- Lower leg -->
-	<property name="xcom_lowerleg" value="0.12185"/>
-	<property name="ycom_lowerleg" value="0.00058"/>
-	<property name="zcom_lowerleg" value="-0.00012"/>
-	<property name="m_lowerleg" value="0.80669"/>
-	<property name="ixx_lowerleg" value="0.00042"/>
-	<property name="iyy_lowerleg" value="0.02202"/>
-	<property name="izz_lowerleg" value="0.02183"/>
-	<property name="ixy_lowerleg" value="0.0"/>
-	<property name="ixz_lowerleg" value="0.0"/>
-	<property name="iyz_lowerleg" value="0.0"/>
+	<xacro:property name="xcom_lowerleg" value="0.12185"/>
+	<xacro:property name="ycom_lowerleg" value="0.00058"/>
+	<xacro:property name="zcom_lowerleg" value="-0.00012"/>
+	<xacro:property name="m_lowerleg" value="0.80669"/>
+	<xacro:property name="ixx_lowerleg" value="0.00042"/>
+	<xacro:property name="iyy_lowerleg" value="0.02202"/>
+	<xacro:property name="izz_lowerleg" value="0.02183"/>
+	<xacro:property name="ixy_lowerleg" value="0.0"/>
+	<xacro:property name="ixz_lowerleg" value="0.0"/>
+	<xacro:property name="iyz_lowerleg" value="0.0"/>
 </robot>

File: urdfs/leg/leg.urdf.xacro (robot description, xacro)
@@ -10,5 +10,5 @@
 		<!-- Slider joint -->
 		<joint name="slider_joint" type="prismatic">
-			<insert_block name="origin"/>
+			<xacro:insert_block name="origin"/>
 			<parent link="${parent}"/>
 			<child  link="trunk"/>

Commit message: [bullet] Added the material information for all the bodies
This information is interpreted by bullet engine

File: urdfs/common.xacro (robot description, xacro)
@@ -52,3 +52,10 @@
 	<property name="ixz_lowerleg" value="0.0"/>
 	<property name="iyz_lowerleg" value="0.0"/>
+    <!-- Materials -->
+    <material name="black">
+      <color rgba="0 0 0 1"/>
+    </material>
+    <material name="grey">
+      <color rgba="0.45 0.45 0.45 1"/>
+    </material>
 </robot>

File: urdfs/leg/leg.urdf.xacro (robot description, xacro)
@@ -65,4 +65,5 @@
 					<mesh filename="package://hyl_description/meshes/leg/trunk.dae" scale="1 1 1"/>
 				</geometry>
+				<material name="grey"/>
 			</visual>
 			<collision>
@@ -86,4 +87,5 @@
 					<mesh filename="package://hyl_description/meshes/leg/hipassembly.dae" scale="1 1 1"/>
 				</geometry>
+				<material name="grey"/>
 			</visual>
 			<collision>
@@ -107,4 +109,5 @@
 					<mesh filename="package://hyl_description/meshes/leg/upperleg.dae" scale="1 1 1"/>
 				</geometry>
+				<material name="grey"/>
 			</visual>
 			<collision>
@@ -127,5 +130,5 @@
 					<mesh filename="package://hyl_description/meshes/leg/lowerleg.dae" scale="1 1 1"/>
 				</geometry>
-				<material name="white"/>
+				<material name="grey"/>
 			</visual>
 			<collision>
@@ -142,4 +145,11 @@
 				<inertia ixx="0.0" iyy="0.0" izz="0.0" ixy="0.0" ixz="0.0" iyz="0.0"/>
 			</inertial>
+			<visual>
+				<origin xyz="0 0 0" rpy="0 0 0"/>
+				<geometry>
+					<sphere radius="0.02185"/>
+				</geometry>
+				<material name="black"/>
+			</visual>
 			<collision>
 				<origin xyz="0 0 0" rpy="0 0 0"/>
